File: schematic/Balancing_robot.kicad_sch (KiCad schematic)
At the start: 34 parts, among them J1 Conn_01x03_Pin, J14 UART2, M1 Motor1, M2 Motor2, SW2 DEBUG[BLUE], U1 STM32F103RBT6, U2 MPU6050, U3 ESP32, U8 L293DD

Commit message: Update README(schematic)
Other:
- note removed: "All 64 ohm resister replaced to 68 ohm"
Changed lines of the file:
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@@
-		)
-	)
-	(text "All 64 ohm resister replaced to 68 ohm"
-		(exclude_from_sim no)
-		(at 185.166 20.066 0)
-		(effects
-			(font
-				(size 1.27 1.27)
-			)
 		)
 	)
