File: schematic/CPU_BLOCK.kicad_sch (KiCad schematic)
At the start: 10 parts, among them J10 SWD, J8 Boot1_Conn, J9 Boot0_Conn, SW3 RESET, Y1 Crystal 8Mh/18pF

Commit message: Update README(schematic)
Other:
- note added: "1,2 connected : SRAM when BOOT0 = 0 2,3 connected : run the program (default)"
- note added: "1,2 connected : system memory / SRAM 2,3 connected : main flash memory (default)"
- note removed: "1,2 connected : main flash memory (default) 2,3 connected : system memory"
- note removed: "1,2 connected : program the device via usb 2,3 connected : run the program (default)"
Changed lines of the file:
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@@
 		)
 	)
-	(text "1,2 connected : main flash memory (default)\n2,3 connected : system memory"
+	(text "1,2 connected : system memory / SRAM\n2,3 connected : main flash memory (default)"
 		(exclude_from_sim no)
 		(at 39.878 72.898 0)
@@
 		)
 	)
-	(text "1,2 connected : program the device via usb\n2,3 connected : run the program (default)"
+	(text "1,2 connected : SRAM when BOOT0 = 0\n2,3 connected : run the program (default)"
 		(exclude_from_sim no)
 		(at 38.608 110.998 0)
