File: schematic/POWER_sch.kicad_sch (KiCad schematic)
At the start: 24 parts, among them J4 10118194-0001LF, J5 PW_Conn, J6 PwSelectPin, J7 Power_conn, U4 LD39050PU33R, U5 L7805CDT-TR

Commit message: Update README(schematic)
Other:
- moved on the sheet: J4, R10, R11, R9
